File: futro-s740-poe.kicad_sch (KiCad schematic)
At the start: 3 parts, among them J1 Conn_02x08, U1 AG5412

Commit message: finished schematics
Signed-off-by: Takuto Nagami <logica0419@gmail.com>
Parts:
- removed J1: Conn_02x08, symbol Connector_Generic:Conn_02x08_Top_Bottom
- added C1: 10nF, Capacitor_SMD:C_1206_3216Metric, symbol Device:C
- added C2: 470μF/16V, Capacitor_THT:CP_Radial_D8.0mm_P3.50mm, symbol Device:C_Polarized
- added D1, D2: MB110S, Package_TO_SOT_SMD:TO-269AA, symbol Diode_Bridge:ABS2
- added J1, J2: Conn_02x08, Connector_PinSocket_2.54mm:PinSocket_2x08_P2.54mm_Vertical_SMD, symbol Connector_Generic:Conn_02x08_Odd_Even
- added U1: SM51589PEL, SM51589PEL:SM51589PEL, symbol SM51589PEL:SM51589PEL
- LED1: renamed from D1; value LED -> Red; footprint (none) -> LED_SMD:LED_0805_2012Metric
- renumbered U1 to U2
Connections:
- net at U2.1 (VIN+): now also LED1.2 (A), C1.1, D1.1 (+), D2.1 (+)
- net at U2.10 (-VDC), U2.7 (-VDC), U2.9 (ADJ): now also C2.2, J2.5 (Pin_5), J2.6 (Pin_6), J2.7 (Pin_7), J2.8 (Pin_8)
- net at U2.2 (VIN-): now also C1.2, D1.2 (-), D2.2 (-)
- net at U2.8 (+VDC): now also C2.1, J2.1 (Pin_1), J2.2 (Pin_2), J2.3 (Pin_3), J2.4 (Pin_4)
- new net: J1.1 (Pin_1), U1.2 (MX1+)
- new net: J1.10 (Pin_10), U1.17 (TD3+)
- new net: J1.11 (Pin_11), U1.9 (MX3-)
- new net: J1.12 (Pin_12), U1.16 (TD3-)
- new net: J1.13 (Pin_13), U1.11 (MX4+)
- new net: J1.14 (Pin_14), U1.14 (TD4+)
- new net: J1.15 (Pin_15), U1.12 (MX4-)
- new net: J1.16 (Pin_16), U1.13 (TD4-)
- new net: J1.2 (Pin_2), U1.23 (TD1+)
- new net: J1.3 (Pin_3), U1.3 (MX1-)
- new net: J1.4 (Pin_4), U1.22 (TD1-)
- new net: J1.5 (Pin_5), U1.5 (MX2+)
- new net: J1.6 (Pin_6), U1.20 (TD2+)
- new net: J1.7 (Pin_7), U1.6 (MX2-)
- new net: J1.8 (Pin_8), U1.19 (TD2-)
- new net: J1.9 (Pin_9), U1.8 (MX3+)
- new net: D2.3, U1.7 (MCT3)
- new net: D2.4, U1.10 (MCT4)
- new net: D1.3, U1.1 (MCT1)
- new net: D1.4, U1.4 (MCT2)
- no-connect marks 0 -> 12
Other:
- note added: "RJ45 Pin 1"
- note added: "RJ45 Pin 2"
- note added: "RJ45 Pin 3"
- note added: "RJ45 Pin 4"
- note added: "RJ45 Pin 5"
- note added: "RJ45 Pin 6"
- note added: "RJ45 Pin 7"
- note added: "RJ45 Pin 8"
- moved on the sheet: LED1, U2

Commit message: migrated to new structure
Signed-off-by: Takuto Nagami <logica0419@gmail.com>
Parts:
- J1, J2: footprint Connector_PinSocket_2.54mm:PinSocket_2x08_P2.54mm_Vertical_SMD -> Connector_PinSocket_2.00mm:PinSocket_2x08_P2.00mm_Vertical_SMD
Changed lines of the file:
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@@
 			)
 		)
-		(property "Footprint" "Connector_PinSocket_2.54mm:PinSocket_2x08_P2.54mm_Vertical_SMD"
+		(property "Footprint" "Connector_PinSocket_2.00mm:PinSocket_2x08_P2.00mm_Vertical_SMD"
 			(at 67.31 33.02 0)
 			(hide yes)
@@
 			)
 		)
-		(property "Footprint" "Connector_PinSocket_2.54mm:PinSocket_2x08_P2.54mm_Vertical_SMD"
+		(property "Footprint" "Connector_PinSocket_2.00mm:PinSocket_2x08_P2.00mm_Vertical_SMD"
 			(at 158.75 104.14 0)
 			(hide yes)
